File: hardware/PUTM_EV_VOLTAGE_INDICATOR_2024.kicad_sch (KiCad schematic)
At the start: 30 parts, among them J1 WIRE, J10 WIRE, J11 SCREW_TERMINAL, J12 SCREW_TERMINAL, J13 WIRE, J14 WIRE, J15 PCB_PAD, J16 PCB_PAD, J17 PCB_PAD, J18 WIRE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

Commit message: esf correction
Connections:
- net at U1.1 (+): now also R2.2, R3.1; no longer RD1.3
- new net: RD1.3, U1.3 (-)
Other:
- moved on the sheet: R2, R3
Changed lines of the file:
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@@
 	)
 	(junction
-		(at 189.23 114.3)
+		(at 189.23 109.22)
 		(diameter 0)
 		(color 0 0 0 0)
@@
 	(wire
 		(pts
-			(xy 194.31 109.22) (xy 196.85 109.22)
+			(xy 189.23 109.22) (xy 189.23 111.76)
+		)
+		(stroke
+			(width 0)
+			(type default)
+		)
+	)
+	(wire
+		(pts
+			(xy 189.23 109.22) (xy 196.85 109.22)
 		)
 		(stroke
@@
 	(wire
 		(pts
-			(xy 189.23 99.06) (xy 189.23 106.68)
+			(xy 189.23 99.06) (xy 189.23 101.6)
 		)
 		(stroke
@@
 	(wire
 		(pts
-			(xy 189.23 121.92) (xy 189.23 124.46)
+			(xy 189.23 116.84) (xy 189.23 124.46)
 		)
 		(stroke
@@
 	(wire
 		(pts
-			(xy 194.31 53.34) (xy 194.31 109.22)
-		)
-		(stroke
-			(width 0)
-			(type default)
-		)
-	)
-	(wire
-		(pts
-			(xy 189.23 114.3) (xy 189.23 116.84)
+			(xy 194.31 53.34) (xy 194.31 114.3)
+		)
+		(stroke
+			(width 0)
+			(type default)
+		)
+	)
+	(wire
+		(pts
+			(xy 189.23 106.68) (xy 189.23 109.22)
 		)
 		(stroke
@@
 	(wire
 		(pts
-			(xy 189.23 111.76) (xy 189.23 114.3)
+			(xy 194.31 114.3) (xy 196.85 114.3)
 		)
 		(stroke
@@
 		(pts
 			(xy 73.66 124.46) (xy 93.98 124.46)
-		)
-		(stroke
-			(width 0)
-			(type default)
-		)
-	)
-	(wire
-		(pts
-			(xy 189.23 114.3) (xy 196.85 114.3)
 		)
 		(stroke
@@
 	(symbol
 		(lib_id "Device:R_Small")
-		(at 189.23 109.22 0)
+		(at 189.23 104.14 0)
 		(unit 1)
 		(exclude_from_sim no)
@@
 		(dnp no)
 		(property "Reference" "R2"
-			(at 185.42 107.95 0)
+			(at 185.42 102.87 0)
 			(effects
 				(font
@@
 		)
 		(property "Value" "67k"
-			(at 185.42 110.49 0)
+			(at 185.42 105.41 0)
 			(effects
 				(font
@@
 		)
 		(property "Footprint" ""
-			(at 189.23 109.22 0)
+			(at 189.23 104.14 0)
 			(effects
 				(font
@@
 		)
 		(property "Datasheet" "~"
-			(at 189.23 109.22 0)
+			(at 189.23 104.14 0)
 			(effects
 				(font
@@
 		)
 		(property "Description" "Resistor, small symbol"
-			(at 189.23 109.22 0)
+			(at 189.23 104.14 0)
 			(effects
 				(font
@@
 	(symbol
 		(lib_id "Device:R_Small")
-		(at 189.23 119.38 0)
+		(at 189.23 114.3 0)
 		(unit 1)
 		(exclude_from_sim no)
@@
 		(dnp no)
 		(property "Reference" "R3"
-			(at 185.42 118.11 0)
+			(at 185.42 113.03 0)
 			(effects
 				(font
@@
 		)
 		(property "Value" "1k"
-			(at 185.42 120.65 0)
+			(at 185.42 115.57 0)
 			(effects
 				(font
@@
 		)
 		(property "Footprint" ""
-			(at 189.23 119.38 0)
+			(at 189.23 114.3 0)
 			(effects
 				(font
@@
 		)
 		(property "Datasheet" "~"
-			(at 189.23 119.38 0)
+			(at 189.23 114.3 0)
 			(effects
 				(font
@@
 		)
 		(property "Description" "Resistor, small symbol"
-			(at 189.23 119.38 0)
-			(effects
-				(font
+			(at 189.23 114.3 0)
+			(effects
+				(font
