File: hardware/PUTM_EV_VOLTAGE_INDICATOR_2024.kicad_pcb (KiCad board)
At the start: 2 copper layers, 60 x 30 mm, 13 parts, among them J11 PCB_PAD, J12 PCB_PAD, J15 PCB_PAD, J16 PCB_PAD, J17 PCB_PAD, J20 PCB_PAD, U1 LM321

Commit message: comparator fix
Parts:
- removed the G*** at (120.0, 67.0)
- removed U1: LM321, Package_TO_SOT_SMD:SOT-23-5
- added U2: LM397, Package_TO_SOT_SMD:SOT-23-5, F.Cu at (129.2, 65.0)
- moved G*** 4.02 mm to (120.4, 60.0)
Routing:
- net /GND: track 31.7 -> 1.19 mm, vias 2 -> 1
- net /HV_MES: track 27.3 -> 25.3 mm, vias 0 -> 2
Other:
- board text removed: "{dblquote}Laziness is such an ugly word, I prefer selective participation.{dblquote}"
